File: SHEM/JCEC/Interface_1.kicad_sch (KiCad schematic)
At the start: 31 parts, among them SW3 SW_Push_SPDT, SW5 SW_Push_SPDT, SW9 SW_Push_SPDT, U11 L78M05CV, U12 TL081, U13 TL081, U14 TL081, U15 TL081

Commit message: maj des schémas
Parts:
- removed R19: R, symbol Device:R
- removed U14: TL081, symbol Amplifier_Operational:TL081
- added D6: 1N4148, Diode_SMD:D_SOD-523, symbol Diode:1N4148WT
- added R65: 3.3K, symbol Device:R
- added U20: TL081, symbol Amplifier_Operational:TL081
- C4: value 1µ / 2,2µ / 10µ -> 100µF
- R1: value R -> 10K
- R19: value R -> 47K
- R2, R20: value R -> 1K
- R20: value R -> 3.3K
- R33: value R -> 100K
- RV10: value R_Potentiometer_Trim -> 10K
- RV11, RV6, RV8: value R_Potentiometer -> 100K
Connections:
- net VCC: now also R33.1, R65.1; no longer R33.2
- net decay_Out_1: now also U20.2 (-), U20.6; no longer C4.1, D1.1 (K), RV1.1, U15.2 (-)
- net at D10.1 (K), RV10.2: now also R33.2; no longer R33.1
- net at R2.1, U13.2 (-): now also R65.2
- net at D10.2 (A), R20.2, RV10.1: now also D6.2 (A)
- net AMP_Piezzo In renamed AMP_Piezzo Out
- net AMP_Piezzo Out: now also D6.1 (K)
- new net: C4.1, D1.1 (K), RV1.1, U15.2 (-), U20.3 (+)
- no-connect marks 6 -> 4
Other:
- note added: "Piezzo to CV"
- note removed: "Piezzo to 3.3V"
- moved on the sheet: D10, RV10
