File: SHEM/JCEC/Interface_2.kicad_sch (KiCad schematic)
At the start: 31 parts, among them SW1 SW_Push_SPDT, SW2 SW_Push_SPDT, SW4 SW_Push_SPDT, U4 L78M05CV, U5 TL081, U6 TL081, U8 TL081, U9 TL081

Commit message: maj des schémas
Parts:
- removed D4: 1N4148, Diode_THT:D_DO-35_SOD27_P7.62mm_Horizontal, symbol Diode:1N4148
- added D4: 1N4148, Diode_SMD:D_SOD-523, symbol Diode:1N4148WT
- added D7: 1N4148, Diode_THT:D_DO-35_SOD27_P7.62mm_Horizontal, symbol Diode:1N4148
- C8: value 1µ / 2,2µ / 10µ -> 100µF
- R13, R18: value R -> 3.3K
- R14: value R -> 10K
- R15, R17: value R -> 1K
- R16: value R -> 47K
- R21: value R -> 100K
- RV2: value R_Potentiometer_Trim -> 10K
- RV3, RV4, RV5: value R_Potentiometer -> 100K
Connections:
- net GND: now also R15.2; no longer R14.2
- net Piezzo In: now also R14.1; no longer R13.1
- net VCC: now also R13.1, R21.1; no longer R21.2, U9.7 (V+)
- net VEE: no longer U9.4 (V-)
- net at R13.2, R15.1: now also U6.2 (-); no longer U5.3 (+)
- net at R17.1, U5.6: now also R16.2; no longer R15.2
- net at D3.2 (A), U6.6: no longer R16.1
- net at D5.2 (A): now also R17.2, RV2.1, D4.2 (A); no longer U9.6
- net at RV2.2: now also D5.1 (K), R21.2; no longer R21.1
- net AMP_Piezzo In: no longer names the net of U8.2 (-), U9.3 (+)
- net AMP_Piezzo In: now also C8.1, RV7.1, D7.1 (K); no longer U6.3 (+), U8.6
- removed net decay_Out_2: C8.1, D5.1 (K), RV7.1, U9.2 (-)
- new net: R14.2, R16.1, U5.3 (+)
- new net: D7.2 (A), U8.6
- new net AMP_Piezzo Out: D4.1 (K), U6.3 (+), U8.3 (+)
- new net decay_Out_1: U9.2 (-), U9.6
Other:
- note added: "Piezzo to CV"
- note removed: "Piezzo to 3.3V"
