File: SHEM/JCEC/stm32_boite_noire.kicad_sch (KiCad schematic)
At the start: 45 parts, among them U10 TL084, U16 TL084, U17 TL084, U18 TL084, U19 TL084

Commit message: maj des schémas
Parts:
- R23, R26, R30, R35, R36, R37, R39, R40, R41, R43, R44, R45, R47, R48, R49, R51, R52, R53, R55, R56, R57, R59, R60: value R -> 10K
- R24, R28, R32, R38, R42, R46, R50, R54, R58: value R -> 3.3K
Connections:
- net GND: now also U16.10 (+), U16.12 (+), U16.3 (+), U16.5 (+), U17.10 (+), U17.12 (+), U17.3 (+), U17.5 (+), U18.10 (+), U18.12 (+), U18.3 (+), U18.5 (+), U19.10 (+), U19.12 (+), U19.3 (+), U19.5 (+)
Other:
- moved on the sheet: R57, R59
